File: trackpad.kicad_sch (KiCad schematic)
At the start: 0 parts

Commit message: Cleanup libraries
Other:
- note added: "TODO controller: Reset button? Testpoints? TODO trackpad: Nothing"
- note removed: "TODO controller: Reset button? Testpoints? ZeoZero ohm resistor to disable 5V line on the VIK header. TODO trackpad: Zero ohm resistor and jumper to toggle use of 5v/3.3v Power. Reset circuit to delay output from LDO. Adjust reset delay on touch controller to be > 90ns after the LDO starts."
Changed lines of the file:
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@@
     (fill (type none))
   )
-  (text "TODO controller:\nReset button?\nTestpoints?\nZeoZero ohm resistor to disable 5V line on the VIK header.\n\nTODO trackpad:\nZero ohm resistor and jumper to toggle use of 5v/3.3v Power.\nReset circuit to delay output from LDO.\nAdjust reset delay on touch controller to be > 90ns after the LDO starts."
+  (text "TODO controller:\nReset button?\nTestpoints?\n\nTODO trackpad:\nNothing"
     (at 306.07 109.22 0)
     (effects (font (size 1.27 1.27)) (justify left bottom))
