File: sensor.kicad_sch (KiCad schematic)
At the start: 36 parts, among them J10 Conn_01x01_Pin, J5 Conn_01x07_Pin, J8 Conn_01x08_Pin, U3 MIC5504-3.3YM5

Commit message: Minor tweaks
Parts:
- C29: LCSC C1525 -> C52923
- R10: LCSC C25744 -> C25752
- R15: LCSC (none) -> C25104
Changed lines of the file:
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@@
+      (effects (font (size 1.27 1.27)) hide)
+    )
+    (property "LCSC" "C25104" (at 196.85 86.36 0)
       (effects (font (size 1.27 1.27)) hide)
     )
@@
       (effects (font (size 1.27 1.27)) hide)
     )
-    (property "LCSC" "C1525" (at 226.06 34.2963 0)
+    (property "LCSC" "C52923" (at 226.06 34.2963 0)
       (effects (font (size 1.27 1.27)) hide)
     )
@@
       (effects (font (size 1.27 1.27)) hide)
     )
-    (property "LCSC" "C1525" (at 180.34 35.56 0)
+    (property "LCSC" "C52923" (at 180.34 35.56 0)
       (effects (font (size 1.27 1.27)) hide)
     )
@@
       (effects (font (size 1.27 1.27)) hide)
     )
-    (property "LCSC" "C25744" (at 55.88 123.19 0)
-      (effects (font (size 1.27 1.27)) hide)
-    )
+    (property "LCSC" "C25752" (at 55.88 123.19 0)
+      (effects (font (size 1.27 1.27)) hide)
+    )
